Commit message: Load Panda dynamics from Franka xacro data

File: rtb-data/rtbdata/xacro/franka_description/robots/hand.xacro (robot description, xacro)
@@ -11,4 +11,9 @@
     </xacro:unless>
     <link name="${ns}_hand">
+      <inertial>
+        <origin xyz="-0.0000376 0.0119128 0.0207260" rpy="0 0 0"/>
+        <mass value="0.6544"/>
+        <inertia ixx="0.00186" ixy="0.00000" ixz="0.00000" iyy="0.00030" iyz="-0.00002" izz="0.00174"/>
+      </inertial>
       <visual>
         <geometry>
@@ -54,4 +59,9 @@
     </link>
     <link name="${ns}_leftfinger">
+      <inertial>
+        <origin xyz="0 0.0152850 0.0219675" rpy="0 0 0"/>
+        <mass value="0.0291"/>
+        <inertia ixx="0.00000849" ixy="0.00000000" ixz="0.00000000" iyy="0.00000853" iyz="-0.00000106" izz="0.00000177"/>
+      </inertial>
       <visual>
         <geometry>
@@ -61,4 +71,9 @@
     </link>
     <link name="${ns}_rightfinger">
+      <inertial>
+        <origin xyz="0 0.0152850 0.0219675" rpy="0 0 0"/>
+        <mass value="0.0291"/>
+        <inertia ixx="0.00000849" ixy="0.00000000" ixz="0.00000000" iyy="0.00000853" iyz="-0.00000106" izz="0.00000177"/>
+      </inertial>
       <visual>
         <origin xyz="0 0 0" rpy="0 0 ${pi}"/>

File: rtb-data/rtbdata/xacro/franka_description/robots/panda_arm.xacro (robot description, xacro)
@@ -12,4 +12,9 @@
     </xacro:unless>
     <link name="${arm_id}_link0">
+      <inertial>
+        <origin xyz="-0.0172 0.0004 0.0745" rpy="0 0 0"/>
+        <mass value="2.3966"/>
+        <inertia ixx="0.0090" ixy="0.0000" ixz="0.0020" iyy="0.0115" iyz="0.0000" izz="0.0085"/>
+      </inertial>
       <visual>
         <geometry>
@@ -37,4 +42,9 @@
     </link>
     <link name="${arm_id}_link1">
+      <inertial>
+        <origin xyz="0.00033 -0.02204 -0.04762" rpy="0 0 0"/>
+        <mass value="2.7907"/>
+        <inertia ixx="0.01564782655" ixy="0.00000531236" ixz="-0.00003676721" iyy="0.01439883526" iyz="-0.00248480843" izz="0.00500443991"/>
+      </inertial>
       <visual>
         <geometry>
@@ -70,4 +80,9 @@
     </joint>
     <link name="${arm_id}_link2">
+      <inertial>
+        <origin xyz="0.00038 -0.09211 0.01908" rpy="0 0 0"/>
+        <mass value="2.5420"/>
+        <inertia ixx="0.01662427728" ixy="0.00003086077" ixz="0.00000835940" iyy="0.00462501261" iyz="0.00355899830" izz="0.01545124526"/>
+      </inertial>
       <visual>
         <geometry>
@@ -103,4 +118,9 @@
     </joint>
     <link name="${arm_id}_link3">
+      <inertial>
+        <origin xyz="0.05152 0.01696 -0.02971" rpy="0 0 0"/>
+        <mass value="2.2513"/>
+        <inertia ixx="0.00631741992" ixy="0.00097309955" ixz="0.00292525834" iyy="0.00866285493" iyz="0.00093469224" izz="0.00657804051"/>
+      </inertial>
       <visual>
         <geometry>
@@ -136,4 +156,9 @@
     </joint>
     <link name="${arm_id}_link4">
+      <inertial>
+        <origin xyz="-0.05113 0.05825 0.01698" rpy="0 0 0"/>
+        <mass value="2.2037"/>
+        <inertia ixx="0.00784585566" ixy="-0.00339591957" ixz="0.00158704074" iyy="0.00649543136" iyz="-0.00181477884" izz="0.01003079917"/>
+      </inertial>
       <visual>
         <geometry>
@@ -169,4 +194,9 @@
     </joint>
     <link name="${arm_id}_link5">
+      <inertial>
+        <origin xyz="-0.00005 0.03730 -0.09280" rpy="0 0 0"/>
+        <mass value="2.2855"/>
+        <inertia ixx="0.02297014781" ixy="-0.00000949345" ixz="-0.00002063156" iyy="0.02095060919" iyz="0.00382345782" izz="0.00430606551"/>
+      </inertial>
       <visual>
         <geometry>
@@ -220,4 +250,9 @@
     </joint>
     <link name="${arm_id}_link6">
+      <inertial>
+        <origin xyz="0.06572 -0.00371 0.00153" rpy="0 0 0"/>
+        <mass value="1.353"/>
+        <inertia ixx="0.00087964522" ixy="-0.00021487814" ixz="-0.00011911662" iyy="0.00277796968" iyz="0.00001274322" izz="0.00286701969"/>
+      </inertial>
       <visual>
         <geometry>
@@ -253,4 +288,9 @@
     </joint>
     <link name="${arm_id}_link7">
+      <inertial>
+        <origin xyz="0.00089 -0.00044 0.05491" rpy="0 0 0"/>
+        <mass value="0.35973"/>
+        <inertia ixx="0.00019541063" ixy="0.00000165231" ixz="0.00000148826" iyy="0.00019210361" iyz="-0.00000131132" izz="0.00017936256"/>
+      </inertial>
       <visual>
         <geometry>
